File: panel-control.sch (KiCad schematic (older format))
At the start: 63 parts, among them J1 POWER_CONN, J2 SWIM, J3 PWR, J4 40HAT, J5 HUB-75_A, J6 HUB-75_B, J7 VBAT, J8 FAN, Q1 DMMT5401, Q2 DMG2305UX, Q3 AO4407A, Q4 S8050, SW1 POW, SW2 NRST, U1 TXS0108EPW, U2 TXS0108EPW, U3 TXS0108EPW, U4 HT7533-1, U5 STM8S103F3P

Commit message: start laying traces
Parts:
- removed C13, C15: 100nF, Capacitor_SMD:C_0603_1608Metric, symbol Device:C
- removed C14: 1uF, Capacitor_SMD:C_0603_1608Metric_Pad1.08x0.95mm_HandSolder, symbol Device:C
- removed MK2: ICS-43434, user_footprints:I2S-MIC_DIP-6, symbol panel-control-rescue:ICS-43434-ICS-43434_DIP-6
- added J9: MK_R, Connector_FFC-FPC:Molex_200528-0060_1x06-1MP_P1.00mm_Horizontal, symbol Connector:Conn_01x06_Female
Connections:
- net BUT_PWR is gone; now on net BUT_POW: J1.2 (Pin_2)
- net +3.3VA: now also J9.1 (Pin_1), J9.2 (Pin_2)
- net G1A_B: now also J5.2 (Pin_2)
- net G1B_B: no longer J5.2 (Pin_2)
- net G2A_B: now also J5.6 (Pin_6)
- net G2B_B: no longer J5.6 (Pin_6)
- net GND: now also J9.6 (Pin_6)
- net M_SCK: now also J9.4 (Pin_4)
- net M_SD: now also J9.5 (Pin_5)
- net M_WS: now also J9.3 (Pin_3)
Changed lines of the file:
@@
-$EndComp
-$Comp
-L panel-control-rescue:ICS-43434-ICS-43434_DIP-6 MK2
-U 1 1 5FB3249C
-P 13800 8500
-F 0 "MK2" H 13800 9167 50  0000 C CNN
-F 1 "ICS-43434" H 13800 9076 50  0000 C CNN
-F 2 "user_footprints:I2S-MIC_DIP-6" H 13800 8500 50  0001 L BNN
-F 3 "" H 13800 8500 50  0001 L BNN
-F 4 "2.43 USD" H 13800 8500 50  0001 L BNN "PRICE"
-F 5 "Bad" H 13800 8500 50  0001 L BNN "AVAILABILITY"
-F 6 "Multi-Mode Microphone with I2S Digital Output" H 13800 8500 50  0001 L BNN "DESCRIPTION"
-F 7 "TDK-InvenSense" H 13800 8500 50  0001 L BNN "MF"
-F 8 "ICS-43434" H 13800 8500 50  0001 L BNN "MP"
-F 9 "LGA-6 TDK-InvenSense" H 13800 8500 50  0001 L BNN "PACKAGE"
-	1    13800 8500
-	1    0    0    -1
 $EndComp
 $Comp
@@
 $EndComp
 $Comp
-L power:+3.3VA #PWR037
-U 1 1 5FB3A0CC
-P 14300 7450
-F 0 "#PWR037" H 14300 7300 50  0001 C CNN
-F 1 "+3.3VA" H 14315 7623 50  0000 C CNN
-F 2 "" H 14300 7450 50  0001 C CNN
-F 3 "" H 14300 7450 50  0001 C CNN
-	1    14300 7450
-	1    0    0    -1
-$EndComp
-$Comp
 L power:GND #PWR028
 U 1 1 5FB3A81B
@@
 $EndComp
 $Comp
-L power:GND #PWR038
-U 1 1 5FB3AE44
-P 14300 9150
-F 0 "#PWR038" H 14300 8900 50  0001 C CNN
-F 1 "GND" H 14300 9000 50  0000 C CNN
-F 2 "" H 14300 9150 50  0000 C CNN
-F 3 "" H 14300 9150 50  0000 C CNN
-	1    14300 9150
-	1    0    0    -1
-$EndComp
-$Comp
 L Device:C C6
 U 1 1 5FB3FADD
@@
 Wire Wire Line
 	11750 8700 11750 8950
-$Comp
-L Device:C C14
-U 1 1 5FB432B4
-P 14300 8500
-F 0 "C14" H 14415 8546 50  0000 L CNN
-F 1 "1uF" H 14415 8455 50  0000 L CNN
-F 2 "Capacitor_SMD:C_0603_1608Metric_Pad1.08x0.95mm_HandSolder" H 14338 8350 50  0001 C CNN
-F 3 "~" H 14300 8500 50  0001 C CNN
-	1    14300 8500
-	1    0    0    -1
-$EndComp
-Wire Wire Line
-	14300 8350 14300 8100
-Connection ~ 14300 8100
-Wire Wire Line
-	14300 8100 14300 7800
-Wire Wire Line
-	14300 8650 14300 8900
-Connection ~ 14300 8900
-Wire Wire Line
-	13000 8300 13300 8300
 Text Label 10300 8300 0    50   ~ 0
 M_WS
-Text Label 13100 8500 0    50   ~ 0
+Text Label 13200 8150 0    50   ~ 0
 M_WS
 Text Label 10300 8400 0    50   ~ 0
@@
 Text Label 10300 8500 0    50   ~ 0
 M_SD
-Text Label 13100 8600 0    50   ~ 0
+Text Label 13200 8250 0    50   ~ 0
 M_SCK
-Text Label 13100 8700 0    50   ~ 0
+Text Label 13200 8350 0    50   ~ 0
 M_SD
 Wire Wire Line
@@
 Wire Wire Line
 	10300 8400 10750 8400
-Wire Wire Line
-	13100 8500 13300 8500
-Wire Wire Line
-	13100 8600 13300 8600
-Wire Wire Line
-	13100 8700 13300 8700
 Text Label 4150 1950 0    50   ~ 0
 M_SCK
@@
 STB_B
 Text Label 5350 5650 0    50   ~ 0
-G2B_B
+G2A_B
 Text Label 5350 5550 0    50   ~ 0
 GND
 Text Label 5350 5450 0    50   ~ 0
-G1B_B
+G1A_B
 Text Label 4000 5450 0    50   ~ 0
 R1A_B
@@
 Wire Wire Line
 	10750 8100 10300 8100
-Wire Wire Line
-	14300 8900 14300 9150
-Wire Wire Line
-	14300 7800 13000 7800
-Wire Wire Line
-	13000 7800 13000 8300
-Connection ~ 14300 7800
-Wire Wire Line
-	14300 7800 14300 7450
 Text Notes 10600 8000 0    50   ~ 0
 Left
-Text Notes 13150 8200 0    50   ~ 0
-Right
 $Comp
 L Device:R R11
@@
 U 1 1 60089960
 P 13850 1650
-F 0 "C12" H 13736 1604 50  0000 R CNN
-F 1 "100nF" H 13736 1695 50  0000 R CNN
+F 0 "C12" H 14100 1600 50  0000 R CNN
+F 1 "100nF" H 14200 1700 50  0000 R CNN
 F 2 "Capacitor_SMD:C_0603_1608Metric" H 13888 1500 50  0001 C CNN
 F 3 "~" H 13850 1650 50  0001 C CNN
@@
 Text Label 5350 6600 0    50   ~ 0
 G1B_B
-Text Label 4000 6600 0    50   ~ 0
-R1B_B
 Text Label 4000 6700 0    50   ~ 0
 B1B_B
@@
 NoConn ~ 7450 7950
 NoConn ~ 7450 8050
-Connection ~ 13850 1500
-Connection ~ 13850 1800
-$Comp
-L Device:C C15
-U 1 1 6008A6B7
-P 14350 1650
-F 0 "C15" H 14236 1604 50  0000 R CNN
-F 1 "100nF" H 14236 1695 50  0000 R CNN
-F 2 "Capacitor_SMD:C_0603_1608Metric" H 14388 1500 50  0001 C CNN
-F 3 "~" H 14350 1650 50  0001 C CNN
-	1    14350 1650
-	1    0    0    1
-$EndComp
-Wire Wire Line
-	14100 1500 14350 1500
-Wire Wire Line
-	13850 1500 14100 1500
-Connection ~ 14100 1500
-Wire Wire Line
-	14100 1800 14350 1800
-Wire Wire Line
-	13850 1800 14100 1800
-Connection ~ 14100 1800
-$Comp
-L Device:C C13
-U 1 1 6008A024
-P 14100 1650
-F 0 "C13" H 13986 1604 50  0000 R CNN
-F 1 "100nF" H 13986 1695 50  0000 R CNN
-F 2 "Capacitor_SMD:C_0603_1608Metric" H 14138 1500 50  0001 C CNN
-F 3 "~" H 14100 1650 50  0001 C CNN
-	1    14100 1650
-	1    0    0    1
-$EndComp
 $Comp
 L Device:LED D1
@@
 $EndComp
 Text Label 1650 7950 0    50   ~ 0
-BUT_PWR
+BUT_POW
 $Comp
 L power:GND #PWR04
@@
 Wire Wire Line
 	4250 9700 4250 9900
+$Comp
+L Connector:Conn_01x06_Female J9
+U 1 1 60033554
+P 13700 8150
+F 0 "J9" H 13728 8126 50  0000 L CNN
+F 1 "MK_R" H 13728 8035 50  0000 L CNN
+F 2 "Connector_FFC-FPC:Molex_200528-0060_1x06-1MP_P1.00mm_Horizontal" H 13700 8150 50  0001 C CNN
+F 3 "~" H 13700 8150 50  0001 C CNN
+	1    13700 8150
+	1    0    0    -1
+$EndComp
+$Comp
+L power:+3.3VA #PWR037
+U 1 1 60036E16
+P 13500 7950
+F 0 "#PWR037" H 13500 7800 50  0001 C CNN
+F 1 "+3.3VA" H 13515 8123 50  0000 C CNN
+F 2 "" H 13500 7950 50  0001 C CNN
+F 3 "" H 13500 7950 50  0001 C CNN
+	1    13500 7950
+	1    0    0    -1
+$EndComp
+$Comp
+L power:GND #PWR038
+U 1 1 600376CF
+P 13500 8450
+F 0 "#PWR038" H 13500 8200 50  0001 C CNN
+F 1 "GND" H 13500 8300 50  0000 C CNN
+F 2 "" H 13500 8450 50  0000 C CNN
+F 3 "" H 13500 8450 50  0000 C CNN
+	1    13500 8450
+	1    0    0    -1
+$EndComp
+Wire Wire Line
+	13500 8050 13350 8050
+Wire Wire Line
+	13350 8050 13350 7950
+Wire Wire Line
+	13350 7950 13500 7950
+Connection ~ 13500 7950
+Wire Wire Line
+	13200 8350 13500 8350
+Wire Wire Line
+	13200 8250 13500 8250
+Wire Wire Line
+	13500 8150 13200 8150
+Text Notes 12950 7900 0    50   ~ 0
+Right
+Text Label 4000 6600 0    50   ~ 0
+R1B_B
 $EndSCHEMATC

Commit message: sort of finished layout
Connections:
- net RST is gone; now on net NRST: J2.4 (Pin_4)
- net +3.3VA: no longer J3.1 (Pin_1), J3.3 (Pin_3)
- net +3V3: now also J3.1 (Pin_1)
- net +5VA: now also J3.3 (Pin_3)
Changed lines of the file:
@@
 Text Label 1100 7150 0    60   ~ 0
 P5V
-Text Label 1100 7050 0    60   ~ 0
-P3V3_HAT
 Wire Wire Line
 	1100 7050 1750 7050
@@
 Wire Wire Line
 	4950 6600 5350 6600
-Text Label 1100 6950 0    60   ~ 0
-P3V3_HAT
 Text Label 1100 7250 0    60   ~ 0
 P5V
@@
 Wire Wire Line
 	2250 7250 2250 7350
-Wire Wire Line
-	1100 6950 1750 6950
 Wire Wire Line
 	1100 7250 1750 7250
@@
 	1350 9750 1500 9750
 Text Label 1500 9850 0    50   ~ 0
-RST
+NRST
 Wire Wire Line
 	1350 9850 1500 9850
@@
 Text Label 4000 6600 0    50   ~ 0
 R1B_B
+Text Label 1100 7050 0    60   ~ 0
+P5V
+$Comp
+L power:+3V3 #PWR0101
+U 1 1 5FFA1320
+P 1750 6950
+F 0 "#PWR0101" H 1750 6800 50  0001 C CNN
+F 1 "+3V3" H 1765 7123 50  0000 C CNN
+F 2 "" H 1750 6950 50  0001 C CNN
+F 3 "" H 1750 6950 50  0001 C CNN
+	1    1750 6950
+	1    0    0    -1
+$EndComp
 $EndSCHEMATC
