File: panel-control.sch (KiCad schematic (older format))
At the start: 60 parts, among them J1 POWER_CONN, J2 SWIM, J3 PWR, J4 40HAT, J5 HUB-75_A, J6 HUB-75_B, J7 VBAT, J8 FAN, J9 MK_R, Q1 DMMT5401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

Commit message: nearly ready to submit
Parts:
- added C13: 1uf, Capacitor_SMD:C_1206_3216Metric, symbol Device:C
- J1: footprint Connector_PinHeader_2.54mm:PinHeader_1x06_P2.54mm_Vertical -> Connector_FFC-FPC:Molex_200528-0060_1x06-1MP_P1.00mm_Horizontal
- Q3: footprint SOIC127P600X175-8N -> libraries:SOIC127P600X175-8N
- R1, R10, R12, R13, R15, R16, R17, R18, R19, R2, R3, R4, R8, R9: footprint Resistor_SMD:R_0603_1608Metric -> Resistor_SMD:R_0402_1005Metric
- R11: footprint Resistor_SMD:R_0603_1608Metric_Pad0.98x0.95mm_HandSolder -> Resistor_SMD:R_0402_1005Metric
- R7: footprint Capacitor_SMD:C_0603_1608Metric_Pad1.08x0.95mm_HandSolder -> Capacitor_SMD:C_0402_1005Metric
Connections:
- wire segments 261 -> 263
Other:
- moved on the sheet: Q1A, Q1B, Q2, R5, R6

Commit message: tweaks to components
Parts:
- C1, C2, C3, C4: footprint Capacitor_SMD:C_0603_1608Metric_Pad1.08x0.95mm_HandSolder -> Capacitor_SMD:C_0603_1608Metric; LCSC (none) -> C14663
- C10, C7: LCSC (none) -> C15849
- C11, C12, C5, C9: LCSC (none) -> C14663
- C6: footprint Capacitor_SMD:C_0603_1608Metric_Pad1.08x0.95mm_HandSolder -> Capacitor_SMD:C_0603_1608Metric; LCSC (none) -> C15849
- C8: footprint Resistor_SMD:R_0603_1608Metric -> Capacitor_SMD:C_0603_1608Metric; LCSC (none) -> C15849
- Q4: LCSC (none) -> C2146
- R1, R2: value 470 -> 330; LCSC (none) -> C25104
- R10, R17, R18, R19: LCSC (none) -> C25744
- R11: value 100K -> 47k; LCSC (none) -> C25792
- R12, R13, R15, R8, R9: LCSC (none) -> C25900
- R14: footprint Resistor_SMD:R_0603_1608Metric -> Resistor_SMD:R_0402_1005Metric; LCSC (none) -> C25900
- R16: value 39k -> 47k; LCSC (none) -> C25792
- R3, R4: value 270 -> 330; LCSC (none) -> C25104
- R5: footprint Resistor_SMD:R_0603_1608Metric_Pad0.84x1.00mm_HandSolder -> Resistor_SMD:R_0402_1005Metric; LCSC (none) -> C25792
- R6: footprint Resistor_SMD:R_0603_1608Metric_Pad0.84x1.00mm_HandSolder -> Resistor_SMD:R_0402_1005Metric; LCSC (none) -> C25744
- R7: footprint Capacitor_SMD:C_0402_1005Metric -> Resistor_SMD:R_0402_1005Metric; LCSC (none) -> C25900
- U1, U2, U3: LCSC (none) -> C17206
Changed lines of the file:
@@
 F 0 "R6" V 6830 3500 50  0000 C CNN
 F 1 "10K" V 6750 3500 50  0000 C CNN
-F 2 "Resistor_SMD:R_0603_1608Metric_Pad0.84x1.00mm_HandSolder" V 6680 3500 50  0001 C CNN
+F 2 "Resistor_SMD:R_0402_1005Metric" V 6680 3500 50  0001 C CNN
 F 3 "" H 6750 3500 50  0001 C CNN
+F 4 "C25744" V 6750 3500 50  0001 C CNN "LCSC"
 	1    6750 3500
 	-1   0    0    -1
@@
 F 0 "R5" V 6030 3500 50  0000 C CNN
 F 1 "47K" V 5950 3500 50  0000 C CNN
-F 2 "Resistor_SMD:R_0603_1608Metric_Pad0.84x1.00mm_HandSolder" V 5880 3500 50  0001 C CNN
+F 2 "Resistor_SMD:R_0402_1005Metric" V 5880 3500 50  0001 C CNN
 F 3 "" H 5950 3500 50  0001 C CNN
+F 4 "C25792" V 5950 3500 50  0001 C CNN "LCSC"
 	1    5950 3500
 	-1   0    0    -1
@@
 F 0 "C2" H 7965 4446 50  0000 L CNN
 F 1 "100nF" H 7965 4355 50  0000 L CNN
-F 2 "Capacitor_SMD:C_0603_1608Metric_Pad1.08x0.95mm_HandSolder" H 7888 4250 50  0001 C CNN
+F 2 "Capacitor_SMD:C_0603_1608Metric" H 7888 4250 50  0001 C CNN
 F 3 "~" H 7850 4400 50  0001 C CNN
+F 4 "C14663" H 7850 4400 50  0001 C CNN "LCSC"
 	1    7850 4400
 	1    0    0    -1
@@
 F 0 "R7" V 7500 4750 50  0000 L CNN
 F 1 "4.7K" V 7600 4700 50  0000 L CNN
-F 2 "Capacitor_SMD:C_0402_1005Metric" V 7530 4800 50  0001 C CNN
+F 2 "Resistor_SMD:R_0402_1005Metric" V 7530 4800 50  0001 C CNN
 F 3 "~" H 7600 4800 50  0001 C CNN
+F 4 "C25900" V 7600 4800 50  0001 C CNN "LCSC"
 	1    7600 4800
 	1    0    0    -1
@@
 F 0 "C6" H 11865 8346 50  0000 L CNN
 F 1 "1uF" H 11865 8255 50  0000 L CNN
-F 2 "Capacitor_SMD:C_0603_1608Metric_Pad1.08x0.95mm_HandSolder" H 11788 8150 50  0001 C CNN
+F 2 "Capacitor_SMD:C_0603_1608Metric" H 11788 8150 50  0001 C CNN
 F 3 "~" H 11750 8300 50  0001 C CNN
+F 4 "C15849" H 11750 8300 50  0001 C CNN "LCSC"
 	1    11750 8300
 	1    0    0    -1
@@
 F 2 "Package_SO:TSSOP-20_4.4x6.5mm_P0.65mm" H 8300 6900 50  0001 C CNN
 F 3 "www.ti.com/lit/ds/symlink/txs0108e.pdf" H 8300 7550 50  0001 C CNN
+F 4 "C17206" H 8300 7650 50  0001 C CNN "LCSC"
 	1    8300 7650
 	1    0    0    -1
@@
 P 10550 8800
 F 0 "R11" H 10620 8846 50  0000 L CNN
-F 1 "100K" H 10620 8755 50  0000 L CNN
+F 1 "47k" H 10620 8755 50  0000 L CNN
 F 2 "Resistor_SMD:R_0402_1005Metric" V 10480 8800 50  0001 C CNN
 F 3 "~" H 10550 8800 50  0001 C CNN
+F 4 "C25792" H 10550 8800 50  0001 C CNN "LCSC"
 	1    10550 8800
 	1    0    0    -1
@@
 F 2 "Capacitor_SMD:C_0603_1608Metric" H 13638 1500 50  0001 C CNN
 F 3 "~" H 13600 1650 50  0001 C CNN
+F 4 "C14663" H 13600 1650 50  0001 C CNN "LCSC"
 	1    13600 1650
 	1    0    0    1
@@
 F 2 "Capacitor_SMD:C_0603_1608Metric" H 13888 1500 50  0001 C CNN
 F 3 "~" H 13850 1650 50  0001 C CNN
+F 4 "C14663" H 13850 1650 50  0001 C CNN "LCSC"
 	1    13850 1650
 	1    0    0    1
@@
 F 0 "R14" H 11870 2846 50  0000 L CNN
 F 1 "4.7k" H 11870 2755 50  0000 L CNN
-F 2 "Resistor_SMD:R_0603_1608Metric" V 11730 2800 50  0001 C CNN
+F 2 "Resistor_SMD:R_0402_1005Metric" V 11730 2800 50  0001 C CNN
 F 3 "~" H 11800 2800 50  0001 C CNN
+F 4 "C25900" H 11800 2800 50  0001 C CNN "LCSC"
 	1    11800 2800
 	1    0    0    -1
@@
 F 2 "Resistor_SMD:R_0402_1005Metric" V 11480 2800 50  0001 C CNN
 F 3 "~" H 11550 2800 50  0001 C CNN
+F 4 "C25900" H 11550 2800 50  0001 C CNN "LCSC"
 	1    11550 2800
 	1    0    0    -1
@@
 F 0 "C8" H 12085 4104 50  0000 R CNN
 F 1 "1uF" H 12085 4195 50  0000 R CNN
-F 2 "Resistor_SMD:R_0603_1608Metric" H 12238 4000 50  0001 C CNN
+F 2 "Capacitor_SMD:C_0603_1608Metric" H 12238 4000 50  0001 C CNN
 F 3 "~" H 12200 4150 50  0001 C CNN
+F 4 "C15849" H 12200 4150 50  0001 C CNN "LCSC"
 	1    12200 4150
 	1    0    0    1
@@
 P 14450 2950
 F 0 "R16" H 14520 2996 50  0000 L CNN
-F 1 "39k" H 14520 2905 50  0000 L CNN
+F 1 "47k" H 14520 2905 50  0000 L CNN
 F 2 "Resistor_SMD:R_0402_1005Metric" V 14380 2950 50  0001 C CNN
 F 3 "~" H 14450 2950 50  0001 C CNN
+F 4 "C25792" H 14450 2950 50  0001 C CNN "LCSC"
 	1    14450 2950
 	1    0    0    -1
@@
 F 2 "Resistor_SMD:R_0402_1005Metric" V 14380 3250 50  0001 C CNN
 F 3 "~" H 14450 3250 50  0001 C CNN
+F 4 "C25744" H 14450 3250 50  0001 C CNN "LCSC"
 	1    14450 3250
 	1    0    0    -1
@@
 F 2 "Capacitor_SMD:C_0603_1608Metric" H 12088 1500 50  0001 C CNN
 F 3 "~" H 12050 1650 50  0001 C CNN
+F 4 "C15849" H 12050 1650 50  0001 C CNN "LCSC"
 	1    12050 1650
 	1    0    0    -1
@@
 F 2 "Capacitor_SMD:C_0603_1608Metric" H 12888 1500 50  0001 C CNN
 F 3 "~" H 12850 1650 50  0001 C CNN
+F 4 "C15849" H 12850 1650 50  0001 C CNN "LCSC"
 	1    12850 1650
 	1    0    0    -1
@@
 P 5000 9150
 F 0 "R3" V 5207 9150 50  0000 C CNN
-F 1 "270" V 5116 9150 50  0000 C CNN
+F 1 "330" V 5116 9150 50  0000 C CNN
 F 2 "Resistor_SMD:R_0402_1005Metric" V 4930 9150 50  0001 C CNN
 F 3 "~" H 5000 9150 50  0001 C CNN
+F 4 "C25104" V 5000 9150 50  0001 C CNN "LCSC"
 	1    5000 9150
 	0    1    -1   0
@@
 P 5000 9700
 F 0 "R4" V 5207 9700 50  0000 C CNN
-F 1 "270" V 5116 9700 50  0000 C CNN
+F 1 "330" V 5116 9700 50  0000 C CNN
 F 2 "Resistor_SMD:R_0402_1005Metric" V 4930 9700 50  0001 C CNN
 F 3 "~" H 5000 9700 50  0001 C CNN
+F 4 "C25104" V 5000 9700 50  0001 C CNN "LCSC"
 	1    5000 9700
 	0    1    -1   0
@@
 F 2 "Package_TO_SOT_SMD:SOT-23" H 9350 1975 50  0001 L CIN
 F 3 "http://www.unisonic.com.tw/datasheet/S8050.pdf" H 9150 2050 50  0001 L CNN
+F 4 "C2146" H 9150 2050 50  0001 C CNN "LCSC"
 	1    9150 2050
 	-1   0    0    -1
@@
 F 2 "Resistor_SMD:R_0402_1005Metric" V 9430 2050 50  0001 C CNN
 F 3 "~" H 9500 2050 50  0001 C CNN
+F 4 "C25900" V 9500 2050 50  0001 C CNN "LCSC"
 	1    9500 2050
 	0    1    1    0
@@
 F 2 "Resistor_SMD:R_0402_1005Metric" V 8980 1700 50  0001 C CNN
 F 3 "~" H 9050 1700 50  0001 C CNN
+F 4 "C25900" V 9050 1700 50  0001 C CNN "LCSC"
 	1    9050 1700
 	-1   0    0    1
@@
 F 2 "Package_SO:TSSOP-20_4.4x6.5mm_P0.65mm" H 8200 9100 50  0001 C CNN
 F 3 "www.ti.com/lit/ds/symlink/txs0108e.pdf" H 8200 9750 50  0001 C CNN
+F 4 "C17206" H 8200 9850 50  0001 C CNN "LCSC"
 	1    8200 9850
 	1    0    0    -1
@@
 F 2 "Resistor_SMD:R_0402_1005Metric" V 9630 2200 50  0001 C CNN
 F 3 "~" H 9700 2200 50  0001 C CNN
+F 4 "C25744" H 9700 2200 50  0001 C CNN "LCSC"
 	1    9700 2200
 	1    0    0    -1
@@
 F 0 "C4" H 9065 4446 50  0000 L CNN
 F 1 "100nF" H 9065 4355 50  0000 L CNN
-F 2 "Capacitor_SMD:C_0603_1608Metric_Pad1.08x0.95mm_HandSolder" H 8988 4250 50  0001 C CNN
+F 2 "Capacitor_SMD:C_0603_1608Metric" H 8988 4250 50  0001 C CNN
 F 3 "~" H 8950 4400 50  0001 C CNN
+F 4 "C14663" H 8950 4400 50  0001 C CNN "LCSC"
 	1    8950 4400
 	1    0    0    -1
@@
 F 2 "Package_SO:TSSOP-20_4.4x6.5mm_P0.65mm" H 8450 4650 50  0001 C CNN
 F 3 "www.ti.com/lit/ds/symlink/txs0108e.pdf" H 8450 5300 50  0001 C CNN
+F 4 "C17206" H 8450 5400 50  0001 C CNN "LCSC"
 	1    8450 5400
 	1    0    0    -1
@@
 F 0 "C3" H 8915 6896 50  0000 L CNN
 F 1 "100nF" H 8915 6805 50  0000 L CNN
-F 2 "Capacitor_SMD:C_0603_1608Metric_Pad1.08x0.95mm_HandSolder" H 8838 6700 50  0001 C CNN
+F 2 "Capacitor_SMD:C_0603_1608Metric" H 8838 6700 50  0001 C CNN
 F 3 "~" H 8800 6850 50  0001 C CNN
+F 4 "C14663" H 8800 6850 50  0001 C CNN "LCSC"
 	1    8800 6850
 	1    0    0    -1
@@
 F 0 "C1" H 7815 8896 50  0000 L CNN
 F 1 "100nF" H 7815 8805 50  0000 L CNN
-F 2 "Capacitor_SMD:C_0603_1608Metric_Pad1.08x0.95mm_HandSolder" H 7738 8700 50  0001 C CNN
+F 2 "Capacitor_SMD:C_0603_1608Metric" H 7738 8700 50  0001 C CNN
 F 3 "~" H 7700 8850 50  0001 C CNN
+F 4 "C14663" H 7700 8850 50  0001 C CNN "LCSC"
 	1    7700 8850
 	-1   0    0    -1
@@
 P 3550 9150
 F 0 "R1" V 3757 9150 50  0000 C CNN
-F 1 "470" V 3666 9150 50  0000 C CNN
+F 1 "330" V 3666 9150 50  0000 C CNN
 F 2 "Resistor_SMD:R_0402_1005Metric" V 3480 9150 50  0001 C CNN
 F 3 "~" H 3550 9150 50  0001 C CNN
+F 4 "C25104" V 3550 9150 50  0001 C CNN "LCSC"
 	1    3550 9150
 	0    -1   -1   0
@@
 P 3550 9700
 F 0 "R2" V 3757 9700 50  0000 C CNN
-F 1 "470" V 3666 9700 50  0000 C CNN
+F 1 "330" V 3666 9700 50  0000 C CNN
 F 2 "Resistor_SMD:R_0402_1005Metric" V 3480 9700 50  0001 C CNN
 F 3 "~" H 3550 9700 50  0001 C CNN
+F 4 "C25104" V 3550 9700 50  0001 C CNN "LCSC"
 	1    3550 9700
 	0    -1   -1   0
@@
 F 2 "Resistor_SMD:R_0402_1005Metric" V 12880 5700 50  0001 C CNN
 F 3 "~" H 12950 5700 50  0001 C CNN
+F 4 "C25900" H 12950 5700 50  0001 C CNN "LCSC"
 	1    12950 5700
 	1    0    0    -1
@@
 F 2 "Capacitor_SMD:C_0603_1608Metric" H 12738 5850 50  0001 C CNN
 F 3 "~" H 12700 6000 50  0001 C CNN
+F 4 "C14663" H 12700 6000 50  0001 C CNN "LCSC"
 	1    12700 6000
 	1    0    0    1
@@
 F 2 "Capacitor_SMD:C_0603_1608Metric" H 11238 5850 50  0001 C CNN
 F 3 "~" H 11200 6000 50  0001 C CNN
+F 4 "C14663" H 11200 6000 50  0001 C CNN "LCSC"
 	1    11200 6000
 	1    0    0    1
@@
 F 2 "Resistor_SMD:R_0402_1005Metric" V 11380 5700 50  0001 C CNN
 F 3 "~" H 11450 5700 50  0001 C CNN
+F 4 "C25900" H 11450 5700 50  0001 C CNN "LCSC"
 	1    11450 5700
 	1    0    0    -1
@@
 F 2 "Resistor_SMD:R_0402_1005Metric" V 14380 4100 50  0001 C CNN
 F 3 "~" H 14450 4100 50  0001 C CNN
+F 4 "C25744" H 14450 4100 50  0001 C CNN "LCSC"
 	1    14450 4100
 	1    0    0    -1
@@
 F 2 "Resistor_SMD:R_0402_1005Metric" V 14380 4400 50  0001 C CNN
 F 3 "~" H 14450 4400 50  0001 C CNN
+F 4 "C25744" H 14450 4400 50  0001 C CNN "LCSC"
 	1    14450 4400
 	1    0    0    -1

Commit message: maybe finished revision with micro usb output
Parts:
- removed J7: VBAT, Connector_PinHeader_2.54mm:PinHeader_1x02_P2.54mm_Vertical, symbol Connector:Conn_01x02_Male
- removed Q1: DMMT5401, Package_TO_SOT_SMD:SOT-23-6, symbol raspberrypi_hat:DMMT5401
- removed Q2: DMG2305UX, Package_TO_SOT_SMD:SOT-23, symbol raspberrypi_hat:DMG2305UX
- removed R5: 47K, Resistor_SMD:R_0402_1005Metric, symbol Device:R
- removed R6: 10K, Resistor_SMD:R_0402_1005Metric, symbol Device:R
- added D5: D, Diode_SMD:D_SMA, symbol Device:D
- added J10: PWR_HAT, Connector_PinHeader_2.54mm:PinHeader_1x02_P2.54mm_Vertical, symbol Connector:Conn_01x02_Male
- added J7: USB_PWR, Connector_USB:USB_Micro-B_Molex-105017-0001, symbol Connector:USB_B_Micro
- C13: value 1uf -> 10uf; LCSC C1848 -> C13585
- J1: footprint Connector_FFC-FPC:Molex_200528-0060_1x06-1MP_P1.00mm_Horizontal -> Connector_FFC-FPC:Molex_200528-0080_1x08-1MP_P1.00mm_Horizontal; symbol Connector:Conn_01x06_Male -> Connector_Generic:Conn_01x08
- J3: footprint Connector_PinHeader_2.54mm:PinHeader_2x04_P2.54mm_Vertical -> Connector_PinHeader_2.54mm:PinHeader_2x03_P2.54mm_Vertical; symbol Connector_Generic:Conn_02x04_Odd_Even -> Connector_Generic:Conn_02x03_Odd_Even
- J9: value MK_R -> I2S; symbol Connector:Conn_01x06_Female -> Connector_Generic:Conn_01x06
Connections:
- net labels added: +5V, +5VP, EXT_POWER, GPIO_POWEROFF, GPIO_SHUTDOWN, USB_PWR
- net labels removed: ID_SC_EEPROM, ID_SD_EEPROM
- wire segments 263 -> 253
- no-connect marks 17 -> 14
Other:
- moved on the sheet: C13

Commit message: better reverse current protection and usb-c power
Parts:
- removed D5: D, Diode_SMD:D_SMA, symbol Device:D
- removed Q3: AO4407A, libraries:SOIC127P600X175-8N, symbol panel-control-rescue:AO4407A-AO4407A
- removed R19: 10k, Resistor_SMD:R_0402_1005Metric, symbol Device:R
- added Q1, Q3: DMG2305UX, Package_TO_SOT_SMD:SOT-23, symbol raspberrypi_hat:DMG2305UX
- added Q2: DMMT5401, Package_TO_SOT_SMD:SOT-23-6, symbol raspberrypi_hat:DMMT5401
- added R5: 4.7k, Resistor_SMD:R_0402_1005Metric, symbol Device:R
- added R6: 10k, Resistor_SMD:R_0402_1005Metric, symbol Device:R
- J7: footprint Connector_USB:USB_Micro-B_Molex-105017-0001 -> Connector_USB:USB_C_Receptacle_GCT_USB4085; symbol Connector:USB_B_Micro -> Connector:USB_C_Plug
- J8: symbol Connector:Conn_01x04_Male -> Connector_Generic:Conn_01x04
- R18: value 10k -> 47k; LCSC C25744 -> (none)
Connections:
- net +3V3: now also R5.1
- net +5V: now also Q1.2 (S), Q2.6 (E), Q3.3 (D)
- net +5VA: now also Q2.5 (E), Q3.2 (S)
- net +5VP: now also J7.A4 (VBUS), J7.A9 (VBUS), J7.B4 (VBUS), J7.B9 (VBUS), Q1.3 (D); no longer J7.1 (VBUS)
- net FAN_TACH: now also U5.20 (PD3), R5.2; no longer R18.1
- net GND: now also J7.A1 (GND), J7.A12 (GND), J7.B1 (GND), J7.B12 (GND), J7.S1 (SHIELD), R18.2, R6.2; no longer J7.5 (GND), J7.6 (Shield)
- net at Q4.3 (C), R8.1: now also Q1.1 (G)
- new net: Q2.1 (C), Q2.2 (B), Q2.3 (B), R6.1
- new net: Q2.4 (C), Q3.1 (G), R18.1
- no-connect marks 14 -> 11
Other:
- note added: "Jumper these to P5B_HAT"
- note removed: "5V Powered HAT Protection"
- note removed: "Check datasheet for amber leds \nto minimize birghtness / current"
- note removed: "I think this is intended to block excessive current\nfrom flowing from the Pi to the Hat, but actually idk.."
- note removed: "This is the recommended 5V rail protection for \na HAT with power going to the Pi.\nSee https://github.com/raspberrypi/hats/blob/master/designguide.md#back-powering-the-pi-via-the-j8-gpio-header"
- moved on the sheet: C13, J10, Q4, R10, R8, R9

Commit message: more revisions, maybe ready to submit
Parts:
- removed C8: 1uF, Capacitor_SMD:C_0603_1608Metric, symbol Device:C
- removed U5: STM8S103F3P, Package_SO:TSSOP-20_4.4x6.5mm_P0.65mm, symbol MCU_ST_STM8:STM8S003F3P
- added J11: BOOT, Connector_PinHeader_2.54mm:PinHeader_1x02_P2.54mm_Vertical, symbol Connector:Conn_01x02_Male
- added R19: 4.7k, Resistor_SMD:R_0402_1005Metric, symbol Device:R
- added R20: 47k, Resistor_SMD:R_0402_1005Metric, symbol Device:R
- added U7: STM32L031F6Px, Package_SO:TSSOP-20_4.4x6.5mm_P0.65mm, symbol MCU_ST_STM32L0:STM32L031F6Px
- C10, C7: value 1uF -> 10uf; LCSC C15849 -> C19702
- C13: footprint Capacitor_SMD:C_1206_3216Metric -> Capacitor_SMD:C_0603_1608Metric; LCSC C13585 -> C19702
- J2: value SWIM -> PROG; footprint Connector_PinHeader_2.54mm:PinHeader_1x04_P2.54mm_Vertical -> Connector_PinHeader_2.54mm:PinHeader_1x06_P2.54mm_Vertical; symbol Connector_Generic:Conn_01x04 -> Connector_Generic:Conn_01x06
- R1, R2, R3, R4: value 330 -> 470; LCSC C25104 -> C25117
- R12, R15: value 4.7k -> 47k
- R13, R14: value 4.7k -> 470; LCSC C25900 -> C25117
- R7: value 4.7K -> 4.7k
Connections:
- net +3V3: now also J2.4 (Pin_4), R19.1, U7.16 (VDD), U7.5 (VDDA); no longer J2.1 (Pin_1), R13.1, R14.1
- net BUT_POW: now also U7.6 (PA0)
- net EXT_POWER: now also U7.14 (PB1)
- net FAN_PWM: now also U7.12 (PA6)
- net FAN_TACH: now also U7.11 (PA5)
- net GND: now also J2.6 (Pin_6), R20.2, U7.15 (VSS); no longer J2.3 (Pin_3)
- net GPIO_POWEROFF: now also U7.3 (PC15)
- net GPIO_SHUTDOWN: now also U7.2 (PC14)
- net I2C_SCL: now also U7.17 (PA9); no longer R14.2
- net I2C_SDA: now also U7.18 (PA10); no longer R13.2
- net LED_BAT: now also U7.20 (PA14)
- net LED_PWR: now also U7.19 (PA13)
- net PWR_EN: now also U7.7 (PA1)
- net at R16.2, R17.1: now also U7.13 (PA7)
- net NRST renamed CTS
- net CTS: now also J2.5 (Pin_5), U7.4 (NRST); no longer J2.4 (Pin_4)
- net SWIM: no longer names the net of J2.2 (Pin_2)
- net SWIM: now also R13.1
- new net: J2.3 (Pin_3), R14.1
- new net: J11.1 (Pin_1), R19.2
- new net BOOT: J11.2 (Pin_2), J2.1 (Pin_1), R20.1, U7.1 (BOOT0)
- new net USART_RX: R13.2, U7.9 (PA3)
- new net USART_TX: R14.2, U7.8 (PA2)
- no-connect marks 11 -> 8
Other:
- moved on the sheet: C5, C9, J8, R12, R15, R16, R17, R5, SW1, SW2

Commit message: finally submitted
Parts:
- removed C2: 100nF, Capacitor_SMD:C_0603_1608Metric, symbol Device:C
- removed U1, U2, U3: TXS0108EPW, Package_SO:TSSOP-20_4.4x6.5mm_P0.65mm, symbol Logic_LevelTranslator:TXS0108EPW
- added R21, R? (x2): 4.7k, Resistor_SMD:R_0402_1005Metric, symbol Device:R
- added U1, U2, U3: 74HC245, Package_SO:SSOP-20_4.4x6.5mm_P0.65mm, symbol 74xx:74HC245
Connections:
- net +3.3VA: no longer C1.1, R7.1
- net +5VA: now also C1.1, R7.2, R21.2, R?.2, R?.2, U1.20 (VCC), U2.20 (VCC), U3.20 (VCC)
- net A_A: now also U1.5 (A3)
- net A_B: now also U1.15 (B3)
- net B1A_A: now also U2.3 (A1)
- net B1A_B: now also U2.17 (B1)
- net B1B_A: now also U3.4 (A2)
- net B1B_B: now also U3.16 (B2)
- net B2A_A: now also U2.6 (A4)
- net B2A_B: now also U2.14 (B4)
- net B2B_A: now also U3.7 (A5)
- net B2B_B: now also U3.13 (B5)
- net B_A: now also U1.6 (A4)
- net B_B: now also U1.14 (B4)
- net CLK_A: now also U1.2 (A0)
- net CLK_B: now also U1.18 (B0)
- net C_A: now also U1.7 (A5)
- net C_B: now also U1.13 (B5)
- net D_A: now also U1.8 (A6)
- net D_B: now also U1.12 (B6)
- net E_A: now also U1.9 (A7)
- net E_B: now also U1.11 (B7)
- net G1A_A: now also U2.4 (A2)
- net G1A_B: now also U2.16 (B2)
- net G1B_A: now also U3.3 (A1)
- net G1B_B: now also U3.17 (B1)
- net G2A_A: now also U2.7 (A5)
- net G2A_B: now also U2.13 (B5)
- net G2B_A: now also U3.6 (A4)
- net G2B_B: now also U3.14 (B4)
- net GND: now also U1.10 (GND), U2.10 (GND), U3.10 (GND)
- net LS_OE: now also R7.1, U1.19 (CE); no longer R7.2
- net OE_A: now also U1.3 (A1)
- net OE_B: now also U1.17 (B1)
- net R1A_A: now also U2.2 (A0)
- net R1A_B: now also U2.18 (B0)
- net R1B_A: now also U3.2 (A0)
- net R1B_B: now also U3.18 (B0)
- net R2A_A: now also U2.5 (A3)
- net R2A_B: now also U2.15 (B3)
- net R2B_A: now also U3.5 (A3)
- net R2B_B: now also U3.15 (B3)
- net STB_A: now also U1.4 (A2)
- net STB_B: now also U1.16 (B2)
- new net: R?.1, U2.19 (CE)
- new net: R?.1, U3.19 (CE)
- new net LS_DIR: R21.1, U1.1 (A->B), U2.1 (A->B), U3.1 (A->B)
Other:
- moved on the sheet: C1, C3, C4, R7
