File: panel-control.kicad_pcb (KiCad board)
At the start: 4 copper layers, 65 x 30 mm, 22 parts, among them J1 PWR, J2 103904-3, J3 40HAT, J4 HUB-75, Q1 DMG2305UX, Q2 DMMT5401, U1 TXS0108EPW, U2 TXS0108EPW

Commit message: update pcb from new sch
Parts:
- added C1: 1uF, Capacitor_SMD:C_0603_1608Metric, F.Cu at (146.7, 97.3)
- added C10: 100nF, Capacitor_SMD:C_0603_1608Metric, F.Cu at (132.1, 95.2)
- added C11: 100nF, Capacitor_SMD:C_0603_1608Metric, F.Cu at (146.7, 92.3)
- added C12: 100nF, Capacitor_SMD:C_0603_1608Metric_Pad1.08x0.95mm_HandSolder, F.Cu at (158.8, 94.0)
- added C15: 100nF, Capacitor_SMD:C_0603_1608Metric_Pad1.08x0.95mm_HandSolder, F.Cu at (119.8, 95.4)
- added C2: 1uF, Capacitor_SMD:C_0603_1608Metric, F.Cu at (151.0, 89.8)
- added C3: 100nF, Capacitor_SMD:C_0603_1608Metric, F.Cu at (170.2, 71.1)
- added C4: 100nF, Capacitor_SMD:C_0603_1608Metric, F.Cu at (170.2, 73.6)
- added C5: 100nF, Capacitor_SMD:C_0603_1608Metric, F.Cu at (165.5, 78.3)
- added C6: 100nF, Capacitor_SMD:C_0603_1608Metric, F.Cu at (160.9, 83.4)
- added C7: 1uF, Resistor_SMD:R_0603_1608Metric, F.Cu at (154.9, 97.8)
- added D1: 5V, LED_SMD:LED_0603_1608Metric, F.Cu at (124.0, 95.4)
- added D2: PWR, LED_SMD:LED_0805_2012Metric, F.Cu at (111.0, 95.0)
- added D3: PI, LED_SMD:LED_0603_1608Metric, F.Cu at (128.1, 95.4)
- added D4: BAT, LED_SMD:LED_0805_2012Metric, F.Cu at (115.4, 95.6)
- added J4: HUB-75_B, user_footprints:TE_5-103167-5, F.Cu at (85.1, 102.9)
- added J6: POWER_CONN, Connector_PinHeader_2.54mm:PinHeader_1x06_P2.54mm_Vertical, F.Cu at (156.6, 72.2)
- added J7: SWIM, Connector_PinHeader_2.54mm:PinHeader_1x04_P2.54mm_Vertical, F.Cu at (161.2, 72.2)
- added Q1: AO4407A, libraries:SOIC127P600X175-8N, F.Cu at (149.3, 85.3)
- added Q2: S8050, Package_TO_SOT_SMD:SOT-23, F.Cu at (154.9, 61.0)
- added R1: 4.7k, Resistor_SMD:R_0603_1608Metric, F.Cu at (155.6, 89.5)
- added R11: 4.7k, Resistor_SMD:R_0603_1608Metric, F.Cu at (159.2, 99.1)
- added R12: 4.7k, Resistor_SMD:R_0603_1608Metric, F.Cu at (146.7, 99.9)
- added R14: 470, Resistor_SMD:R_0603_1608Metric, F.Cu at (159.6, 89.5)
- added R15: 270, Resistor_SMD:R_0603_1608Metric, F.Cu at (150.7, 97.3)
- added R16: 470, Resistor_SMD:R_0603_1608Metric, F.Cu at (148.1, 69.7)
- added R17: 270, Resistor_SMD:R_0603_1608Metric, F.Cu at (154.7, 94.5)
- added R2: 4.7k, Resistor_SMD:R_0603_1608Metric, F.Cu at (150.7, 92.3)
- added R3: 4.7k, Resistor_SMD:R_0603_1608Metric, F.Cu at (146.7, 94.8)
- added R4: 39k, Resistor_SMD:R_0603_1608Metric, F.Cu at (136.1, 95.2)
- added R5: 4.7k, Resistor_SMD:R_0603_1608Metric, F.Cu at (148.1, 67.2)
- added R6: 10k, Resistor_SMD:R_0603_1608Metric, F.Cu at (150.7, 94.8)
- added R7: 10k, Resistor_SMD:R_0603_1608Metric, F.Cu at (174.2, 71.1)
- added SW1: POW, Button_Switch_SMD:SW_Push_1P1T_NO_6x6mm_H9.5mm, F.Cu at (163.8, 110.5)
- added SW2: NRST, Button_Switch_SMD:SW_Push_1P1T_NO_6x6mm_H9.5mm, F.Cu at (151.1, 108.0)
- added U1: HT7533-1, Package_TO_SOT_SMD:SOT-89-3, F.Cu at (171.4, 99.1)
- added U2: STM8S103F3P, Package_SO:TSSOP-20_4.4x6.5mm_P0.65mm, F.Cu at (177.8, 87.6)
- added U5: TXS0108EPW, Package_SO:TSSOP-20_4.4x6.5mm_P0.65mm, F.Cu at (92.7, 92.7)
- C8: renamed from C1; value 1uF -> 100nF
- C9: renamed from C2; value 1uF -> 100nF
- J2: value 103904-3 -> VBAT; footprint user_footprints:TE_103904-3 -> Connector_PinHeader_2.54mm:PinHeader_1x02_P2.54mm_Vertical
- J3: renamed from J4; value HUB-75 -> HUB-75_A
- J5: renamed from J1; footprint Connector_PinHeader_2.54mm:PinHeader_2x02_P2.54mm_Vertical -> Connector_PinHeader_2.54mm:PinHeader_2x04_P2.54mm_Vertical
- moved J2 61.9 mm to (165.8, 72.2), turned to 0 degrees
- moved J5 33.1 mm to (72.4, 86.4)
- moved J3 19.2 mm to (116.8, 102.9)
- renumbered C3 to C13, C4 to C14, J3 to J1, Q1 to Q3, Q2 to Q4, R1 to R10, R3 to R13, R5 to R8, R6 to R9, U1 to U3, U2 to U4
Connections:
- net /B1_A renamed /B1A_A
- net /B1_B renamed /B1A_B
- net /B2_B renamed /B2A_B
- net /G1_A renamed /G1A_A
- net /G2_A renamed /G2A_A
- net /R1_B renamed /R1A_B
- net /R2_B renamed /R2A_B
- J1 pad 10: /OE_A -> /E_A
- J1 pad 19: /SDA_A -> /B2A_A
- J1 pad 22: /D_A -> /R1B_A
- J1 pad 23: /SCL_A -> /R1A_A
- J1 pad 24: /E_A -> /R2A_A
- J1 pad 27: /ID_SD_EEPROM -> (no net)
- J1 pad 28: /ID_SC_EEPROM -> (no net)
- J1 pad 29: /R2_A -> /G1B_A
- J1 pad 3: Net-(J3-Pad3) -> /I2C_SDA
- J1 pad 31: /R1_A -> /B1B_A
- J1 pad 32: Net-(J3-Pad32) -> /OE_A
- J1 pad 33: Net-(J3-Pad33) -> /G2B_A
- J1 pad 36: Net-(J3-Pad36) -> /B2B_A
- J1 pad 37: /B2_A -> /R2B_A
- J1 pad 40: Net-(J3-Pad40) -> (no net)
- J1 pad 5: Net-(J3-Pad5) -> /I2C_SCL
- J1 pad 8: Net-(J3-Pad8) -> /D_A
- J2 pad 1: +5VA -> /VBAT_SENSE
- J2 pad 2: /SDA_B -> GND
- J3 pad 2: /G1_B -> /G1B_B
- J3 pad 6: /G2_B -> /G2B_B
- J5 pad 3: +5VA -> +3.3VA
- Q3 pad 1: Net-(Q1-Pad1) -> Net-(Q3-Pad1)
- Q3 pad 3: +5VA -> /EXT_5V
- Q4 pad 1: Net-(Q2-Pad1) -> Net-(Q3-Pad1)
- Q4 pad 2: Net-(Q2-Pad1) -> Net-(Q4-Pad2)
- Q4 pad 3: Net-(Q2-Pad1) -> Net-(Q4-Pad2)
- Q4 pad 4: Net-(Q1-Pad1) -> Net-(Q4-Pad2)
- Q4 pad 5: /P5V_HAT -> /EXT_5V
- Q4 pad 6: +5VA -> /P5V_HAT
- R8 pad 1: Net-(Q1-Pad1) -> Net-(Q3-Pad1)
- R9 pad 1: Net-(Q2-Pad1) -> Net-(Q4-Pad2)
- U3 pad 1: /SDA_A -> /CLK_A
- U3 pad 12: /C_B -> /E_B
- U3 pad 13: /B_B -> /D_B
- U3 pad 14: /A_B -> /C_B
- U3 pad 15: /STB_B -> /B_B
- U3 pad 16: /OE_B -> /A_B
- U3 pad 17: /CLK_B -> /STB_B
- U3 pad 18: /SCL_B -> /OE_B
- U3 pad 20: /SDA_B -> /CLK_B
- U3 pad 3: /SCL_A -> /OE_A
- U3 pad 4: /CLK_A -> /STB_A
- U3 pad 5: /OE_A -> /A_A
- U3 pad 6: /STB_A -> /B_A
- U3 pad 7: /A_A -> /C_A
- U3 pad 8: /B_A -> /D_A
- U3 pad 9: /C_A -> /E_A
- U4 pad 1: /R1_A -> /R1A_A
- U4 pad 12: /D_B -> (no net)
- U4 pad 13: /E_B -> (no net)
- U4 pad 14: /G2_B -> (no net)
- U4 pad 17: /G1_B -> (no net)
- U4 pad 5: /R2_A -> /R2A_A
- U4 pad 6: /B2_A -> /B2A_A
- U4 pad 8: /E_A -> (no net)
- U4 pad 9: /D_A -> (no net)
Routing:
- net GND: track 110.3 -> 86.9 mm
- net /SDA_B: track 23.0 -> 0.00 mm, vias 1 -> 0
- net /SCL_B: track 18.7 -> 0.00 mm
- net /B_B: track 12.9 -> 0.00 mm, vias 1 -> 0
- net /STB_B: track 12.7 -> 0.00 mm
- net /CLK_B: track 11.8 -> 23.0 mm
- net /A_B: track 11.1 -> 0.00 mm, vias 1 -> 0
- net /G1_B: track 10.7 -> 0.00 mm
- net /G2_B: track 10.2 -> 0.00 mm
- net /D_B: track 9.08 -> 0.00 mm
- net /C_B: track 8.43 -> 0.00 mm
- net /E_B: track 8.40 -> 0.00 mm
- net /OE_B: track 10.9 -> 18.7 mm
- net /R1A_B: track 6.51 -> 0.00 mm
- net /B1A_B: track 6.00 -> 0.44 mm
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
Commit message: add fan connector to sch
Parts:
- added J8: FAN, Connector_PinSocket_2.54mm:PinSocket_1x04_P2.54mm_Vertical, F.Cu at (180.3, 68.6)
- added R18: 10k, Resistor_SMD:R_0603_1608Metric, F.Cu at (184.6, 67.5)
- added R19: 10k, Resistor_SMD:R_0603_1608Metric, F.Cu at (188.6, 67.5)
- renumbered C15 to C1, C2 to C10, C3 to C11, C4 to C12, C5 to C13, C6 to C15, C8 to C2, C12 to C3, C9 to C4, C10 to C5, C13 to C6, C1 to C7, C7 to C8, C11 to C9, D3 to D2, D2 to D3, H3 to H2, H2 to H3, J6 to J1, J7 to J2, J5 to J3, J1 to J4, J3 to J5, J4 to J6, J2 to J7, Q4 to Q1, Q3 to Q2, Q1 to Q3, Q2 to Q4, R14 to R1, R7 to R10, R13 to R11, R11 to R12, R1 to R13, R2 to R14, R12 to R15, R4 to R16, R6 to R17, R16 to R2, R15 to R3, R17 to R4, R8 to R5, R9 to R6, R10 to R7, R3 to R8, R5 to R9, U5 to U1, U4 to U2, U1 to U4, U2 to U5
Connections:
- J1 pad 2: (no net) -> /BUT_PWR
- J2 pad 4: (no net) -> /RST
- J4 pad 27: (no net) -> /ID_SD_EEPROM
- J4 pad 28: (no net) -> /ID_SC_EEPROM
- J4 pad 40: (no net) -> /I2S_OUT
- U1 pad 12: (no net) -> Net-(U1-Pad12)
- U1 pad 13: (no net) -> Net-(U1-Pad13)
- U1 pad 8: (no net) -> Net-(U1-Pad8)
- U1 pad 9: (no net) -> Net-(U1-Pad9)
- U2 pad 12: (no net) -> Net-(U2-Pad12)
- U2 pad 13: (no net) -> Net-(U2-Pad13)
- U2 pad 14: (no net) -> /G2A_B
- U2 pad 17: (no net) -> /G1A_B
- U2 pad 8: (no net) -> Net-(U2-Pad8)
- U2 pad 9: (no net) -> Net-(U2-Pad9)
- U5 pad 1: (no net) -> Net-(U5-Pad1)
- U5 pad 10: (no net) -> Net-(U5-Pad10)
- U5 pad 14: (no net) -> /FAN_PWM
- U5 pad 15: (no net) -> Net-(U5-Pad15)
- U5 pad 16: (no net) -> Net-(U5-Pad16)
- U5 pad 17: (no net) -> Net-(U5-Pad17)
- U5 pad 20: (no net) -> Net-(R18-Pad2)
- U5 pad 6: (no net) -> Net-(U5-Pad6)
Routing:
- net Net-(Q1-Pad1) (its old number): track 6.02 -> 0.00 mm
- net Net-(Q1-Pad1): track 0.00 -> 6.02 mm

Commit message: fix footprints
Parts:
- J5, J6: footprint user_footprints:TE_5-103167-5 -> Connector_IDC:IDC-Header_2x08_P2.54mm_Vertical
- J8: footprint Connector_PinSocket_2.54mm:PinSocket_1x04_P2.54mm_Vertical -> Connector:FanPinHeader_1x04_P2.54mm_Vertical
- moved J8 6.48 mm to (179.1, 74.9)

Commit message: work on new pcb layout
Parts:
- MK2: footprint user_footprints:I2S-MIC_DIP-6 -> Connector_FFC-FPC:Molex_200528-0060_1x06-1MP_P1.00mm_Horizontal
- R1, R18, R19, R2, R9: footprint Resistor_SMD:R_0603_1608Metric -> Resistor_SMD:R_0402_1005Metric
- moved SW1 111.3 mm to (82.8, 34.2), turned to 270 degrees
- moved SW2 95.1 mm to (91.1, 34.2), turned to 90 degrees
- moved U4 91.5 mm to (99.7, 42.3), turned to 90 degrees
- moved U5 89.6 mm to (95.6, 51.8), turned to 180 degrees
- moved R1 84.6 mm to (82.3, 55.0), turned to 90 degrees
- moved C8 71.8 mm to (100.8, 50.6), turned to 90 degrees
- moved Q3 69.7 mm to (86.2, 55.8), turned to 270 degrees
- moved Q4 69.5 mm to (86.4, 49.9), turned to 270 degrees
- moved R2 66.9 mm to (82.3, 57.9), turned to 90 degrees
- moved R9 65.4 mm to (85.8, 47.1), turned to 180 degrees
- moved J6 63.7 mm to (111.0, 44.7), turned to 180 degrees
- moved D4 62.7 mm to (81.0, 43.3), turned to 270 degrees
- moved J8 61.7 mm to (133.6, 33.1)
- moved H2 61.7 mm to (82.0, 25.7)
- moved H4 61.0 mm to (140.2, 26.3)
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Connections:
- D2 pad 1: Net-(D2-Pad1) -> GND
- D4 pad 1: Net-(D2-Pad1) -> GND
- J1 pad 2: /BUT_PWR -> (no net)
- J2 pad 4: /RST -> (no net)
- J4 pad 27: /ID_SD_EEPROM -> (no net)
- J4 pad 28: /ID_SC_EEPROM -> (no net)
- J4 pad 40: /I2S_OUT -> (no net)
- Q1 pad 6: /P5V_HAT -> Net-(Q1-Pad6)
- Q2 pad 2: /P5V_HAT -> Net-(Q1-Pad6)
- Q3 pad 5: /EXT_5V -> /P5V_HAT
- Q3 pad 6: /EXT_5V -> /P5V_HAT
- Q3 pad 7: /EXT_5V -> /P5V_HAT
- Q3 pad 8: /EXT_5V -> /P5V_HAT
- U1 pad 12: Net-(U1-Pad12) -> (no net)
- U1 pad 13: Net-(U1-Pad13) -> (no net)
- U1 pad 8: Net-(U1-Pad8) -> (no net)
- U1 pad 9: Net-(U1-Pad9) -> (no net)
- U2 pad 12: Net-(U2-Pad12) -> (no net)
- U2 pad 13: Net-(U2-Pad13) -> (no net)
- U2 pad 14: /G2A_B -> (no net)
- U2 pad 17: /G1A_B -> (no net)
- U2 pad 8: Net-(U2-Pad8) -> (no net)
- U2 pad 9: Net-(U2-Pad9) -> (no net)
- U5 pad 1: Net-(U5-Pad1) -> (no net)
- U5 pad 10: Net-(U5-Pad10) -> (no net)
- U5 pad 15: Net-(U5-Pad15) -> (no net)
- U5 pad 16: Net-(U5-Pad16) -> (no net)
- U5 pad 17: Net-(U5-Pad17) -> (no net)
- U5 pad 6: Net-(U5-Pad6) -> (no net)
Routing:
- net +3.3VA: track 103.4 -> 0.00 mm, vias 1 -> 0
- net /M_WS: track 92.1 -> 0.00 mm
- net /M_SD: track 90.1 -> 0.00 mm
- net /M_SCK: track 76.3 -> 7.32 mm
- net GND: track 86.9 -> 37.6 mm, vias 1 -> 0
- net /G2A_A: track 41.3 -> 0.00 mm, vias 1 -> 0
- net /G1A_A: track 33.9 -> 0.00 mm, vias 1 -> 0
- net +5VA: track 39.4 -> 5.97 mm
- net /B2_A: track 23.3 -> 0.00 mm
- net /CLK_B: track 23.0 -> 0.00 mm, vias 1 -> 0
- net /LS_OE: track 22.6 -> 0.00 mm
- net /B_A: track 20.3 -> 0.00 mm, vias 1 -> 0
- net /OE_B: track 18.7 -> 0.00 mm
- net /STB_A: track 18.4 -> 0.00 mm, vias 1 -> 0
- net /OE_A: track 17.7 -> 0.00 mm, vias 1 -> 0
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- added copper zone on F.Cu, net (none)
- removed copper zone on F.Cu, net +5VA
- removed copper zone on F.Cu, net GND
Other:
- board size 65 x 30 mm -> 65 x 55.9 mm

Commit message: start laying traces
Parts:
- removed C13, C15: 100nF, Capacitor_SMD:C_0603_1608Metric
- removed MK2: ICS-43434, Connector_FFC-FPC:Molex_200528-0060_1x06-1MP_P1.00mm_Horizontal
- added J9: MK_R, Connector_FFC-FPC:Molex_200528-0060_1x06-1MP_P1.00mm_Horizontal, F.Cu at (138.7, 41.6)
- J1: footprint Connector_PinHeader_2.54mm:PinHeader_1x06_P2.54mm_Vertical -> Connector_FFC-FPC:Molex_200528-0060_1x06-1MP_P1.00mm_Horizontal
- J3, J5, J6, J8: moved to B.Cu
- R10, R12, R13, R15, R16, R17, R3, R4, R8: footprint Resistor_SMD:R_0603_1608Metric -> Resistor_SMD:R_0402_1005Metric
- R11: footprint Resistor_SMD:R_0603_1608Metric_Pad0.98x0.95mm_HandSolder -> Resistor_SMD:R_0402_1005Metric
- R7: footprint Capacitor_SMD:C_0603_1608Metric_Pad1.08x0.95mm_HandSolder -> Capacitor_SMD:C_0402_1005Metric
- moved C5 120.4 mm to (82.8, 39.9), turned to 90 degrees
- moved R16 119.1 mm to (106.1, 24.7)
- moved R4 88.7 mm to (81.0, 45.3), turned to 180 degrees
- moved R10 85.7 mm to (90.2, 54.0), turned to 270 degrees
- moved R3 83.9 mm to (81.0, 50.8), turned to 180 degrees
- moved R17 81.8 mm to (106.1, 26.2), turned to 180 degrees
- moved C9 81.3 mm to (86.9, 37.2), turned to 270 degrees
- moved R8 77.3 mm to (85.0, 48.3)
- moved C12 75.3 mm to (98.7, 50.1)
- moved C11 74.9 mm to (98.7, 48.6)
- moved C1 74.9 mm to (121.6, 57.0), turned to 270 degrees
- moved R12 72.9 mm to (101.0, 55.2), turned to 180 degrees
- moved C7 72.3 mm to (96.1, 45.7), turned to 270 degrees
- moved R13 66.9 mm to (95.6, 60.0), turned to 180 degrees
- moved R14 64.9 mm to (95.2, 58.8), turned to 180 degrees
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Connections:
- J1 pad 2: (no net) -> /BUT_POW
- J2 pad 4: (no net) -> /RST
- J4 pad 27: (no net) -> /ID_SD_EEPROM
- J4 pad 28: (no net) -> /ID_SC_EEPROM
- J4 pad 40: (no net) -> /I2S_OUT
- J5 pad 2: /G1B_B -> /G1A_B
- J5 pad 6: /G2B_B -> /G2A_B
- U1 pad 12: (no net) -> Net-(U1-Pad12)
- U1 pad 13: (no net) -> Net-(U1-Pad13)
- U1 pad 8: (no net) -> Net-(U1-Pad8)
- U1 pad 9: (no net) -> Net-(U1-Pad9)
- U2 pad 12: (no net) -> Net-(U2-Pad12)
- U2 pad 13: (no net) -> Net-(U2-Pad13)
- U2 pad 14: (no net) -> /G2A_B
- U2 pad 17: (no net) -> /G1A_B
- U2 pad 8: (no net) -> Net-(U2-Pad8)
- U2 pad 9: (no net) -> Net-(U2-Pad9)
- U5 pad 1: (no net) -> Net-(U5-Pad1)
- U5 pad 10: (no net) -> Net-(U5-Pad10)
- U5 pad 15: (no net) -> Net-(U5-Pad15)
- U5 pad 16: (no net) -> Net-(U5-Pad16)
- U5 pad 17: (no net) -> Net-(U5-Pad17)
- U5 pad 6: (no net) -> Net-(U5-Pad6)
Routing:
- net +3.3VA: track 0.00 -> 105.2 mm, vias 0 -> 2
- net /M_SCK: track 7.32 -> 59.5 mm
- net /M_SD: track 0.00 -> 49.2 mm
- net /CLK_B: track 0.00 -> 38.6 mm
- net /B2B_B: track 0.00 -> 32.4 mm
- net /M_WS: track 0.00 -> 30.8 mm
- net /R2B_B: track 0.00 -> 29.9 mm
- net /A_B: track 0.00 -> 28.9 mm
- net +3V3: track 0.00 -> 27.5 mm
- net /B1B_B: track 0.00 -> 24.9 mm
- net /E_B: track 0.00 -> 24.5 mm
- net /B_B: track 0.00 -> 24.1 mm
- net /C_B: track 0.00 -> 23.8 mm, vias 0 -> 1
- net /LS_OE: track 0.00 -> 22.7 mm, vias 0 -> 3
- net +5VA: track 5.97 -> 28.1 mm
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- added copper zone on F.Cu, net +5VA
- added copper zone on F.Cu, net /RST
- added copper zone on In1.Cu, net GND
- added copper zone on In2.Cu, net GND
- removed copper zone on F.Cu, net (none)
Other:
- board size 65 x 55.9 mm -> 65 x 45 mm

Commit message: sort of finished layout
Parts:
- removed C14: 1uF, Capacitor_SMD:C_0603_1608Metric_Pad1.08x0.95mm_HandSolder
- removed Q1: DMMT5401, Package_TO_SOT_SMD:SOT-23-6
- removed Q2: DMG2305UX, Package_TO_SOT_SMD:SOT-23
- removed R5: 47K, Resistor_SMD:R_0603_1608Metric_Pad0.84x1.00mm_HandSolder
- removed R6: 10K, Resistor_SMD:R_0603_1608Metric_Pad0.84x1.00mm_HandSolder
- moved R18 17.0 mm to (120.4, 25.3)
- moved R19 17.0 mm to (120.4, 27.6)
- moved R11 9.34 mm to (133.1, 60.6)
- moved J2 8.47 mm to (98.0, 39.3), turned to 180 degrees
- moved J8 7.37 mm to (132.4, 25.9), turned to 180 degrees
- moved R16 2.74 mm to (105.5, 27.4)
- moved R17 2.74 mm to (105.5, 28.9)
- moved J7 2.22 mm to (102.2, 27.1)
- moved R10 1.66 mm to (90.9, 52.6), turned to 90 degrees
- moved C10 1.59 mm to (102.9, 47.7), turned to 270 degrees
- moved R9 0.79 mm to (89.8, 52.6)
- moved R13 0.48 mm to (95.5, 60.5)
- moved C5 0.41 mm to (82.8, 40.3)
- moved C11 0.31 mm to (98.7, 48.3)
- moved R14 0.29 mm to (95.1, 59.1)
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Connections:
- J2 pad 4: /RST -> /NRST
- J3 pad 1: +3.3VA -> +3V3
- J3 pad 3: +3.3VA -> +5VA
Routing:
- net GND: track 37.7 -> 104.8 mm, vias 0 -> 11
- net +5VA: track 28.1 -> 94.6 mm, vias 0 -> 3
- net /FAN_PWM: track 0.00 -> 51.9 mm, vias 0 -> 1
- net Net-(R18-Pad2): track 0.00 -> 48.4 mm, vias 0 -> 2
- net Net-(R16-Pad2): track 0.00 -> 42.7 mm, vias 0 -> 2
- net /NRST: track 10.3 -> 46.9 mm, vias 0 -> 2
- net /BUT_POW: track 15.9 -> 47.5 mm, vias 0 -> 2
- net +3V3: track 27.5 -> 58.8 mm, vias 0 -> 1
- net /LED_PWR: track 19.3 -> 45.8 mm, vias 2 -> 3
- net /SWIM: track 0.00 -> 24.1 mm, vias 0 -> 1
- net /LED_BAT: track 21.3 -> 41.9 mm, vias 2 -> 3
- net +3.3VA: track 105.2 -> 88.2 mm
- net /CLK_B: track 38.6 -> 22.2 mm, vias 0 -> 1
- net /STB_B: track 8.81 -> 22.3 mm
- net /B2B_B: track 32.4 -> 19.0 mm, vias 0 -> 1
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- added copper zone on In2.Cu, net +5VA
- added copper zone on In2.Cu, net /P5V_HAT
- added copper zone on F.Cu, net GND
- removed copper zone on F.Cu, net /RST

Commit message: nearly ready to submit
Parts:
- added C13: 1uf, Capacitor_SMD:C_1206_3216Metric, F.Cu at (90.4, 60.0)
- moved J8 0.07 mm to (132.3, 25.8)
Routing:
- net GND: track 104.8 -> 107.9 mm
- net /I2C_SCL: track 16.6 -> 15.5 mm
- net /I2C_SDA: track 21.3 -> 22.3 mm
Other:
- board text added: "5VA"
- board text added: "A"
- board text added: "B"
- board text added: "BAT"
- board text added: "FAN"
- board text added: "MK_R"
- board text added: "PI"
- board text added: "POW"
- board text added: "POWER_FPC"
- board text added: "RST"
- board text added: "SWIM"
- board text added: "VBAT_SENSE"

Commit message: tweaks to components
Parts:
- R1, R2: value 470 -> 330
- R11: value 100K -> 47k
- R16: value 39k -> 47k
- R3, R4: value 270 -> 330
Changed lines of the file:
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@@
     (34 B.Paste user)
     (35 F.Paste user)
-    (36 B.SilkS user)
-    (37 F.SilkS user)
+    (36 B.SilkS user hide)
+    (37 F.SilkS user hide)
     (38 B.Mask user)
     (39 F.Mask user)
@@
     (fp_line (start 2.3 -1.15) (end 2.3 1.15) (layer F.CrtYd) (width 0.05))
     (fp_line (start 2.3 1.15) (end -2.3 1.15) (layer F.CrtYd) (width 0.05))
-    (pad 2 smd roundrect (at 1.475 0) (size 1.15 1.8) (layers F.Cu F.Paste F.Mask) (roundrect_rratio 0.217391)
+    (pad 2 smd roundrect (at 1.475 0) (size 1.15 1.8) (layers F.Cu F.Paste F.Mask) (roundrect_rratio 0.2173904347826087)
       (net 1 GND))
-    (pad 1 smd roundrect (at -1.475 0) (size 1.15 1.8) (layers F.Cu F.Paste F.Mask) (roundrect_rratio 0.217391)
+    (pad 1 smd roundrect (at -1.475 0) (size 1.15 1.8) (layers F.Cu F.Paste F.Mask) (roundrect_rratio 0.2173904347826087)
       (net 2 /P5V_HAT))
     (model ${KISYS3DMOD}/Capacitor_SMD.3dshapes/C_1206_3216Metric.wrl
@@
       (effects (font (size 1 1) (thickness 0.15)))
     )
-    (fp_text value 100K (at 0 1.43) (layer F.Fab)
+    (fp_text value 47k (at 0 1.43) (layer F.Fab)
       (effects (font (size 1 1) (thickness 0.15)))
     )
@@
       (effects (font (size 1 1) (thickness 0.15)))
     )
-    (fp_text value 39k (at 0 1.43) (layer F.Fab)
+    (fp_text value 47k (at 0 1.43) (layer F.Fab)
       (effects (font (size 1 1) (thickness 0.15)))
     )
@@
       (effects (font (size 1 1) (thickness 0.15)))
     )
-    (fp_text value 270 (at 0 1.43) (layer F.Fab)
+    (fp_text value 330 (at 0 1.43) (layer F.Fab)
       (effects (font (size 1 1) (thickness 0.15)))
     )
@@
       (effects (font (size 1 1) (thickness 0.15)))
     )
-    (fp_text value 270 (at 0 1.43) (layer F.Fab)
+    (fp_text value 330 (at 0 1.43) (layer F.Fab)
       (effects (font (size 1 1) (thickness 0.15)))
     )
@@
       (effects (font (size 1 1) (thickness 0.15)))
     )
-    (fp_text value 470 (at 0 1.43 90) (layer F.Fab)
+    (fp_text value 330 (at 0 1.43 90) (layer F.Fab)
       (effects (font (size 1 1) (thickness 0.15)))
     )
@@
       (effects (font (size 1 1) (thickness 0.15)))
     )
-    (fp_text value 470 (at 0 1.43 90) (layer F.Fab)
+    (fp_text value 330 (at 0 1.43 90) (layer F.Fab)
       (effects (font (size 1 1) (thickness 0.15)))
     )
@@
   (module libraries:SOIC127P600X175-8N (layer F.Cu)
     (at 86.3092 52.959 270)
+    (attr smd)
     (fp_text reference Q3 (at -0.325 -3.635 90) (layer F.SilkS)
       (effects (font (size 1 1) (thickness 0.015)))
